Commit message: added so-101 URDF

File: playground/public/URDF/SO101/arm.urdf (robot description, URDF)
Before this commit: robot so_arm100, 7 links, 6 joints
Links:
- link Base: mass 1.0 -> 0.147; geometry collision mesh filename=meshes/base_motor_holder_so101_v1.stl; collision mesh filename=meshes/base_so101_v2.stl
- link Fixed_Jaw: mass 0.0929859 -> 0.087; geometry collision mesh filename=meshes/sts3215_03a_v1.stl; collision mesh filename=meshes/wrist_roll_follower_so101_v1.stl
- link Lower_Arm: mass 0.147968 -> 0.104; geometry collision mesh filename=meshes/motor_holder_so101_wrist_v1.stl; collision mesh filename=meshes/sts3215_03a_v1.stl
- link Moving_Jaw: mass 0.0202444 -> 0.012; geometry collision mesh filename=meshes/moving_jaw_so101_v1.stl; visual mesh filename=meshes/moving_jaw_so101_v1.stl
- link Rotation_Pitch: mass 0.119226 -> 0.100006; geometry collision mesh filename=meshes/motor_holder_so101_base_v1.stl; collision mesh filename=meshes/rotation_pitch_so101_v1.stl
- link Upper_Arm: mass 0.162409 -> 0.103; geometry collision mesh filename=meshes/sts3215_03a_v1.stl; collision mesh filename=meshes/upper_arm_so101_v1.stl
- link Wrist_Pitch_Roll: mass 0.0661321 -> 0.079; geometry collision mesh filename=meshes/sts3215_03a_no_horn_v1.stl; collision mesh filename=meshes/wrist_roll_pitch_so101_v2.stl
Joints:
- joint Elbow: axis 1 0 0 -> 0 0 1; limit lower=-3.14158 upper=0 effort=35 velocity=1 -> lower=-3.22886 upper=0.0872665 effort=10 velocity=10; origin xyz=0 0.11257 0.028 rpy=1.57079 0 0 -> xyz=-0.11257 -0.028 2.29417e-16 rpy=-2.26208e-15 -1.3739e-15 3.14159
- joint Jaw: limit lower=-0.2 upper=2.0 effort=35 velocity=1 -> lower=-0.261799 upper=1.74533 effort=10 velocity=10; origin xyz=-0.0202 -0.0244 0 rpy=0 3.14158 0 -> xyz=0.0202 0.0188 -0.0234 rpy=1.5708 4.00612e-15 -2.2678e-16
- joint Pitch: axis 1 0 0 -> 0 0 1; limit lower=0 upper=3.5 effort=35 velocity=1 -> lower=-0.174533 upper=3.31613 effort=10 velocity=10; origin xyz=0 0.1025 0.0306 rpy=-1.8 0 0 -> xyz=-0.0303992 -0.0182778 -0.0542 rpy=1.5708 8.18789e-16 3.14159
- joint Rotation: axis 0 1 0 -> 0 0 1; limit lower=-2 upper=2 effort=35 velocity=1 -> lower=-1.91986 upper=1.91986 effort=10 velocity=10; origin xyz=0 -0.0452 0.0165 rpy=1.57079 0 0 -> xyz=0.0207909 -0.0230745 0.0948817 rpy=-3.14159 6.03684e-16 1.5708
- joint Wrist_Pitch: axis 1 0 0 -> 0 0 1; limit lower=-2.5 upper=1.2 effort=35 velocity=1 -> lower=-1.65806 upper=1.65806 effort=10 velocity=10; origin xyz=0 0.0052 0.1349 rpy=-1 0 0 -> xyz=-0.1349 0.0052 3.21791e-16 rpy=-1.11022e-16 1.11022e-16 -1.5708
- joint Wrist_Roll: axis 0 1 0 -> 0 0 1; limit lower=-3.14158 upper=3.14158 effort=35 velocity=1 -> lower=-2.79253 upper=2.79253 effort=10 velocity=10; origin xyz=0 -0.0601 0 rpy=0 1.57079 0 -> xyz=-2.77556e-17 -0.0611 0.0181 rpy=1.5708 2.18394e-16 3.14159

Commit message: centered URDF

File: playground/public/URDF/SO101/arm.urdf (robot description, URDF)
Before this commit: robot so101, 7 links, 6 joints
Joints:
- joint Rotation: origin xyz=0.0207909 -0.0230745 0.0948817 rpy=-3.14159 6.03684e-16 1.5708 -> xyz=0 -0.0452 0.0648 rpy=-3.14159 6.03684e-16 1.5708

Commit message: update rotation axis in urdf

File: playground/public/URDF/SO101/arm.urdf (robot description, URDF)
Before this commit: robot so101, 7 links, 6 joints
Joints:
- joint Rotation: axis 0 0 1 -> 0 0 -1

Commit message: revert to original direction

File: playground/public/URDF/SO101/arm.urdf (robot description, URDF)
Before this commit: robot so101, 7 links, 6 joints
Joints:
- joint Rotation: axis 0 0 -1 -> 0 0 1

Commit message: fix rotation?

File: playground/public/URDF/SO101/arm.urdf (robot description, URDF)
Before this commit: robot so101, 7 links, 6 joints
Joints:
- joint Rotation: origin xyz=0 -0.0452 0.0648 rpy=-3.14159 6.03684e-16 1.5708 -> xyz=0 -0.0452 0.0648 rpy=0 0 1.5708

Commit message: fix rotation - attempt2

File: playground/public/URDF/SO101/arm.urdf (robot description, URDF)
Before this commit: robot so101, 7 links, 6 joints
Joints:
- joint Rotation: origin xyz=0 -0.0452 0.0648 rpy=0 0 1.5708 -> xyz=0 -0.0452 0.0648 rpy=0 0 -1.5708

Commit message: IK visibility toggle

File: playground/public/URDF/SO101/arm.urdf (robot description, URDF)
Before this commit: robot so101, 7 links, 6 joints
Joints:
- joint Rotation: origin xyz=0 -0.0452 0.0648 rpy=0 0 -1.5708 -> xyz=0 -0.0452 0.0648 rpy=-3.14159 6.03684e-16 1.5708
